Commit message: updated version urdf

File: module_3_assignment/urdf/diff_4.urdf (robot description, URDF)
Before this commit: robot mobile_manipulator, 10 links, 9 joints
Links:
- removed link wheel_left_link
- removed link wheel_right_link
- added link back, mass 1; collision box size=0.05 0.04 0.01; visual box size=0.05 0.04 0.01
- added link wheel_back_left_link, mass 2; collision cylinder length=0.1 radius=0.15; visual cylinder length=0.1 radius=0.15
- added link wheel_back_right_link, mass 2; collision cylinder length=0.1 radius=0.15; visual cylinder length=0.1 radius=0.15
- added link wheel_front_left_link, mass 2; collision cylinder length=0.1 radius=0.15; visual cylinder length=0.1 radius=0.15
- added link wheel_front_right_link, mass 2; collision cylinder length=0.1 radius=0.15; visual cylinder length=0.1 radius=0.15
Joints:
- added joint back_joint: type fixed, parent base, child back, origin xyz=0.2 0.0 -0.07 rpy=0.0 0.0 0.0, axis 0 0 1
- added joint wheel_left_joint_b: type continuous, parent back, child wheel_back_left_link, origin xyz=0.2 -0.25 0.0 rpy=1.57 0.0 0.0, axis 0.0 0.0 1.0
- added joint wheel_right_joint_b: type continuous, parent back, child wheel_back_right_link, origin xyz=0.2 0.25 0.0 rpy=1.57 0.0 0.0, axis 0.0 0.0 1.0
- joint finger_joint: origin xyz=0.0 0.0 0.30 rpy=1.57 0.0 0.0 -> xyz=0.0 0.0 0.30 rpy=0.0 0.0 0.0
- joint frame_base_joint: origin xyz=0.0 0.0 0.25 rpy=0.0 0.0 0.0 -> xyz=0.0 0.0 0.25 rpy=0.0 0.0 1.5
- joint frame_down_joint: limit lower=-0.5 upper=0.7 effort=10 velocity=1.0 -> lower=-1.0 upper=0.5 effort=10 velocity=1.0; origin xyz=0.1 0.0 0.25 rpy=1.57 0.0 0.0 -> xyz=0.1 0.0 0.25 rpy=-0.5 0.0 0.0
- joint frame_middle_joint: limit lower=-0.5 upper=0.7 effort=10 velocity=1.0 -> lower=-1.0 upper=0.5 effort=10 velocity=1.0; origin xyz=0.1 0.0 0.25 rpy=1.57 0.0 0.0 -> xyz=0.1 0.0 0.25 rpy=-0.5 0.0 0.0
- joint steering_joint: origin xyz=0.2 0.0 -0.07 rpy=0.0 0.0 0.0 -> xyz=-0.1 0.0 -0.07 rpy=0.0 0.0 0.0
- joint wheel_left_joint: child wheel_left_link -> wheel_front_left_link; origin xyz=0.2 -0.25 0.0 rpy=1.57 0.0 0.0 -> xyz=-0.1 -0.25 0.0 rpy=1.57 0.0 0.0
- joint wheel_right_joint: child wheel_right_link -> wheel_front_right_link; origin xyz=0.2 0.25 0.0 rpy=1.57 0.0 0.0 -> xyz=-0.1 0.25 0.0 rpy=1.57 0.0 0.0

File: module_3_assignment/urdf/manipulator.urdf (robot description, URDF)
Before this commit: robot manipulator, 5 links, 4 joints
Joints:
- joint finger_joint: origin xyz=0.0 0.0 0.30 rpy=1.57 0.0 0.0 -> xyz=0.0 0.0 0.30 rpy=0.0 0.0 0.0
- joint frame_base_joint: origin xyz=0.0 0.0 0.25 rpy=0.0 0.0 0.0 -> xyz=0.0 0.0 0.25 rpy=0.0 0.0 1.5
- joint frame_down_joint: limit lower=-0.5 upper=0.7 effort=10 velocity=1.0 -> lower=-1.0 upper=0.5 effort=10 velocity=1.0; origin xyz=0.1 0.0 0.25 rpy=1.57 0.0 0.0 -> xyz=0.1 0.0 0.25 rpy=-0.5 0.0 0.0
- joint frame_middle_joint: limit lower=-0.5 upper=0.7 effort=10 velocity=1.0 -> lower=-1.0 upper=0.5 effort=10 velocity=1.0; origin xyz=0.1 0.0 0.25 rpy=1.57 0.0 0.0 -> xyz=0.1 0.0 0.25 rpy=-0.5 0.0 0.0
