Commit message: design task3

File: module_5_assignment/urdf/manipulator.urdf (robot description, URDF)
Before this commit: robot manipulator, 5 links, 4 joints
Links:
- removed link base_link
- added link base, mass 1; collision box size=0.75 0.4 0.1; visual box size=0.75 0.4 0.1
Joints:
- joint frame_base_joint: parent base_link -> base

Commit message: task3 success

File: module_5_assignment/urdf/manipulator.urdf (robot description, URDF)
Before this commit: robot manipulator, 5 links, 4 joints
Joints:
- joint frame_base_joint: type continuous -> fixed
